File: 40m_FT8_BD6CR.brd (EAGLE design)
At the start: 147.3 x 107.6 mm, 54 parts, among them IC1 LM7805, IC2 NE602, Q1 2N3904, Q2 2N3904, Q3 2N3904, Q4 BD139, Q5 7074, Q6 7074, X1 JST-XH-02-PIN, X2 JST-XH-02-PIN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

Commit message: updated with vias.
Still some work to do on vias and routing
Parts:
- removed X1, X2, X3: JST-XH-02-PIN, Rembrandt Electronics - JST XH Connectors v1-0:JST-XH-02-PACKAGE-LONG-PAD
- added COAX: 50_Ohm, con-coax:R141426
- added JP2, JP3: (no value), SparkFun-Connectors:AUDIO-JACK
- S1: value DPDT -> DPDT Latching PCB Mount
- moved JP1 48.9 mm to (5.08, 96.5), turned to 0 degrees
- moved D3 34.7 mm to (6.35, 83.8), turned to 90 degrees
- moved LED1 10.9 mm to (50.8, 91.4)
- moved R4 10.2 mm to (59.7, 82.5), turned to 0 degrees
- moved LED2 10.2 mm to (50.8, 77.5), turned to 0 degrees
- moved S1 8.98 mm to (33.0, 95.2)
- moved C10 7.62 mm to (72.4, 83.8)
- moved C11 7.62 mm to (101.6, 82.5)
- moved C12 7.62 mm to (94.0, 82.5)
- moved U$2 7.62 mm to (83.8, 90.2)
- moved U$3 7.62 mm to (111.8, 90.2)
- moved C13 7.62 mm to (120.7, 76.2)
- moved R3 7.18 mm to (78.7, 21.6), turned to 180 degrees
- moved R6 5.24 mm to (90.2, 17.8), turned to 0 degrees
- moved C14 1.27 mm to (138.4, 62.2)
Connections:
- net GND: now also COAX.2, COAX.3, COAX.4, COAX.5, JP2.SLEEVE, JP3.SLEEVE; no longer X1.2, X2.2, X3.2
- net N$27: now also JP2.RING, JP2.TIP; no longer X2.1
- net N$3: now also COAX.1; no longer X3.1
- net N$7: now also JP3.RING, JP3.TIP; no longer X1.1
Routing:
- net 12V: track 7.33 -> 56.7 mm, vias 0 -> 1
- net N$5: track 96.8 -> 63.5 mm
- net N$15: track 64.8 -> 39.4 mm
- net N$27: track 14.2 -> 31.7 mm
- net N$3: track 19.1 -> 35.6 mm
- net N$7: track 12.2 -> 27.1 mm
- net 12V_T: track 14.3 -> 29.0 mm
- net N$26: track 117.8 -> 127.9 mm
- net N$31: track 179.4 -> 169.9 mm
- net N$30: track 33.5 -> 38.7 mm
- net 12V_R: track 20.7 -> 25.4 mm
- net N$17: track 42.5 -> 46.4 mm
- net N$13: track 25.4 -> 26.7 mm
- net N$6: track 7.89 -> 9.12 mm
- net N$10: track 20.8 -> 21.6 mm
Other:
- board size 147.3 x 107.6 mm -> 147.3 x 100 mm

Commit message: Ready for version 1 review
Ready for version 1 review.  Added vias and finished traces on the
bottom side of the board.
Parts:
- moved C2 22.5 mm to (49.5, 59.7), turned to 270 degrees
- moved C3 2.54 mm to (62.2, 55.9)
- moved R1 2.54 mm to (72.4, 55.9)
- moved C13 2.54 mm to (120.7, 78.7)
Routing:
- net 12V_R: track 25.4 -> 114.8 mm, vias 0 -> 1
- net 12V: track 56.7 -> 110.7 mm
- net N$7: track 27.1 -> 61.1 mm
- net N$13: track 26.7 -> 36.8 mm
- net N$3: track 35.6 -> 33.0 mm
- net N$22: track 26.7 -> 24.2 mm
